File: hw/SiPDrive/SiPDrive.kicad_pcb (KiCad board)
At the start: 8 copper layers, 77 parts, among them Q1 SP40N03GNJ, Q2 SP40N03GNJ, Q3 SP40N03GNJ, Q4 SP40N03GNJ, Q5 SP40N03GNJ, Q6 SP40N03GNJ, U1 STSPIN32G4, U2 MT6701, U3 TCAN1057, U4 LDO, U5 SH-3P, U6 SH-3P

Commit message: started routing
Parts:
- removed C6: 100n, Capacitor_SMD:C_0201_0603Metric
- added C18: 10uF, Capacitor_SMD:C_1206_3216Metric, B.Cu at (36.2, 55.8)
- added C19: 10uF, Capacitor_SMD:C_1206_3216Metric, B.Cu at (36.2, 54.0)
- added C20: 10uF, Capacitor_SMD:C_1206_3216Metric, B.Cu at (36.2, 52.2)
- added C21: 10uF, Capacitor_SMD:C_1206_3216Metric, B.Cu at (36.2, 50.3)
- added C22: 10uF, Capacitor_SMD:C_1206_3216Metric, F.Cu at (75.8, 55.0)
- added C23: 10uF, Capacitor_SMD:C_1206_3216Metric, F.Cu at (75.8, 58.4)
- added C3: 100n, Capacitor_SMD:C_0201_0603Metric, F.Cu at (57.5, 63.7)
- added D3: SMBJ26A_C908802, SiPDrive:SMB_L4.5-W3.7-LS5.4-RD, F.Cu at (67.2, 51.3)
- C12, JP1, Q2, Q4, Q6, R1, R19, R21, R3, R5, R6, R8, U2: moved to B.Cu
- C7: footprint Capacitor_SMD:C_0603_1608Metric -> Capacitor_SMD:C_0402_1005Metric
- moved D1 31.5 mm to (52.5, 63.0), turned to 90 degrees
- moved C5 30.3 mm to (63.4, 52.9), turned to 180 degrees
- moved C30 29.4 mm to (55.4, 53.7)
- moved C4 28.6 mm to (61.8, 52.9), turned to 180 degrees
- moved JP1 28.1 mm to (51.5, 80.5), turned to 90 degrees
- moved R14 27.9 mm to (79.3, 77.6)
- moved R21 27.7 mm to (57.8, 50.4), turned to 90 degrees
- moved C7 27.0 mm to (54.7, 60.3), turned to 180 degrees
- moved U1 26.5 mm to (60.6, 58.1), turned to 90 degrees
- moved C1 25.5 mm to (60.1, 52.9), turned to 180 degrees
- moved R19 25.2 mm to (63.9, 50.4), turned to 90 degrees
- moved R1 25.2 mm to (60.8, 50.4), turned to 90 degrees
- moved C9 24.8 mm to (54.8, 65.3), turned to 180 degrees
- moved L1 24.4 mm to (54.5, 62.7), turned to 90 degrees
- moved U6 23.8 mm to (52.9, 57.0), turned to -90 degrees
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Routing:
- net GND: track 0.00 -> 18.6 mm, vias 0 -> 6
- net Net-(Q2-S): track 0.00 -> 16.5 mm, vias 0 -> 2
- net Net-(Q6-S): track 0.00 -> 13.9 mm, vias 0 -> 2
- net Net-(Q4-S): track 0.00 -> 12.8 mm, vias 0 -> 2
- net /PhaseU: track 0.00 -> 7.15 mm, vias 0 -> 15
- net Net-(Q1-G): track 0.00 -> 6.85 mm, vias 0 -> 2
- net /PhaseW: track 0.00 -> 6.59 mm, vias 0 -> 15
- net /PhaseV: track 0.00 -> 6.56 mm, vias 0 -> 15
- net +3.3V: track 0.00 -> 6.47 mm, vias 0 -> 2
- net Net-(Q3-G): track 0.00 -> 6.26 mm, vias 0 -> 2
- net Net-(Q5-G): track 0.00 -> 5.67 mm, vias 0 -> 2
- net +12V: track 0.00 -> 5.17 mm
- net +BATT: track 0.00 -> 4.74 mm
- net Net-(U1-PA7): track 0.00 -> 3.95 mm
- net Net-(U1-SCREF): track 0.00 -> 3.93 mm
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Other:
- board outline added: 20 x 27 mm
- copper layers 8 -> 6

Commit message: Final routing, code fixes, production files and BOM
Parts:
- removed C22, C23: 10uF, Capacitor_SMD:C_1206_3216Metric
- added C24: 10uF, Capacitor_SMD:C_1206_3216Metric, B.Cu at (67.0, 58.2)
- added C25: 10uF, Capacitor_SMD:C_1206_3216Metric, B.Cu at (67.0, 63.7)
- added C26: 10uF, Capacitor_SMD:C_1206_3216Metric, B.Cu at (53.3, 58.4)
- added C32: 10uF, Capacitor_SMD:C_1206_3216Metric, B.Cu at (53.3, 60.2)
- added C33: 10uF, Capacitor_SMD:C_1206_3216Metric, B.Cu at (53.3, 62.0)
- added C34: 10uF, Capacitor_SMD:C_1206_3216Metric, B.Cu at (53.3, 63.9)
- added C35: 10uF, Capacitor_SMD:C_1206_3216Metric, B.Cu at (67.0, 56.4)
- added C36: 10uF, Capacitor_SMD:C_1206_3216Metric, B.Cu at (67.0, 54.5)
- added C37: 10uF, Capacitor_SMD:C_1206_3216Metric, B.Cu at (66.9, 52.8)
- added C6: 10uF, Capacitor_SMD:C_1206_3216Metric, B.Cu at (67.0, 61.9)
- added C8: 10uF, Capacitor_SMD:C_1206_3216Metric, B.Cu at (67.0, 60.1)
- added U7: ~, SiPDrive:SiPDrive_EDGE, F.Cu at (60.8, 58.5)
- C13, C17, TP1, TP2, TP3, TP4, U3, U4: moved to B.Cu
- moved R12 46.1 mm to (58.0, 52.7), turned to 180 degrees
- moved TP4 43.6 mm to (57.5, 61.2), turned to 90 degrees
- moved TP2 41.1 mm to (60.0, 54.8), turned to 90 degrees
- moved TP3 40.5 mm to (60.5, 61.2), turned to 90 degrees
- moved TP1 38.0 mm to (63.0, 54.8), turned to 90 degrees
- moved C15 36.0 mm to (58.0, 51.9)
- moved R11 29.7 mm to (56.8, 52.5), turned to -90 degrees
- moved R6 26.0 mm to (63.0, 57.9)
- moved U2 26.0 mm to (60.7, 58.0)
- moved C12 26.0 mm to (63.0, 56.7)
- moved C16 23.5 mm to (66.4, 63.8), turned to -90 degrees
- moved JP1 22.2 mm to (63.1, 61.5)
- moved R13 21.3 mm to (65.8, 63.9), turned to -90 degrees
- moved U3 20.2 mm to (57.4, 55.2), turned to -90 degrees
- moved C13 18.4 mm to (57.1, 57.5), turned to 0 degrees
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Routing:
- net GND: track 18.6 -> 53.6 mm, vias 6 -> 52
- net +BATT: track 4.74 -> 33.7 mm, vias 0 -> 126
- net /BOARD_NTC: track 0.00 -> 14.8 mm, vias 0 -> 2
- net Net-(U1-GLS1): track 0.37 -> 13.0 mm, vias 1 -> 2
- net /CAN_L: track 0.00 -> 11.0 mm, vias 0 -> 2
- net /CAN_H: track 0.00 -> 10.4 mm, vias 0 -> 1
- net Net-(U1-GLS2): track 0.00 -> 9.51 mm, vias 1 -> 2
- net /SWCLK: track 0.00 -> 7.85 mm, vias 0 -> 1
- net /STATOR_NTC: track 0.00 -> 6.87 mm
- net Net-(U1-GLS3): track 0.07 -> 6.55 mm, vias 1 -> 2
- net +12V: track 5.17 -> 11.3 mm, vias 0 -> 1
- net /BOOT0: track 1.05 -> 6.56 mm, vias 0 -> 1
- net /SWDIO: track 0.00 -> 4.95 mm, vias 0 -> 1
- net +3.3V: track 6.47 -> 11.1 mm, vias 2 -> 9
- net /CAN_RX: track 0.00 -> 4.31 mm, vias 0 -> 1
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- added copper zone on In3.Cu, net +3.3V
- added copper zone on F.Cu, net +BATT
- added copper zone on In2.Cu, net +BATT
- added copper zone on B.Cu, net GND
- added copper zone on In1.Cu, net GND
- added copper zone on In4.Cu, net GND
- added copper zone on B.Cu, net Net-(Q2-S)
- added copper zone on B.Cu, net Net-(Q4-S)
- added copper zone on B.Cu, net Net-(Q6-S)
Other:
- outline, holes or cut-outs redrawn
- board text added: "+"
- board text added: "-"
- board text added: "Boot"
- board text added: "DRIVE"
- board text added: "Mode"
- board text added: "NTC"
- board text added: "RST"
- board text added: "SIP"
- board text added: "SWC"
- board text added: "SWD"
